Commit message: updated xacro joint velocity limits.

File: minima/ros1_gripper/urdf_minima_description/urdf/urdf_minima.xacro (robot description, xacro)
@@ -149,5 +149,5 @@
   <child link="Joint1_v4_1"/>
   <axis xyz="0.0 -0.0 1.0"/>
-  <limit upper="1.570796" lower="-1.570796" effort="100" velocity="10"/>
+  <limit upper="1.570796" lower="-1.570796" effort="100" velocity="6.5"/>
 </joint>
 <joint name="Revolute2" type="revolute">
@@ -156,5 +156,5 @@
   <child link="Joint2_v4_1"/>
   <axis xyz="0.0 1.0 0.0"/>
-  <limit upper="2.96706" lower="0.0" effort="100" velocity="10"/>
+  <limit upper="2.96706" lower="0.0" effort="100" velocity="6.5"/>
 </joint>
 <joint name="Revolute3" type="revolute">
@@ -163,5 +163,5 @@
   <child link="Joint3_v5_1"/>
   <axis xyz="0.0 1.0 0.0"/>
-  <limit upper="6.283185" lower="4.18879" effort="100" velocity="10"/>
+  <limit upper="6.283185" lower="4.18879" effort="100" velocity="6.5"/>
 </joint>
 <joint name="Revolute4" type="revolute">
@@ -170,5 +170,5 @@
   <child link="Joint4_v2_1"/>
   <axis xyz="-0.0 1.0 0.0"/>
-  <limit upper="1.570796" lower="-1.570796" effort="100" velocity="10"/>
+  <limit upper="1.570796" lower="-1.570796" effort="100" velocity="6.5"/>
 </joint>
 <joint name="Slider5" type="prismatic">
@@ -177,5 +177,5 @@
   <child link="Left_jaw_v1_1"/>
   <axis xyz="-0.0 1.0 0.0"/>
-  <limit upper="0.008" lower="0.0" effort="100" velocity="5"/>
+  <limit upper="0.008" lower="0.0" effort="100" velocity="6.5"/>
 </joint>
 <joint name="Slider6" type="prismatic">
@@ -184,5 +184,5 @@
   <child link="Right_jaw_v1_1"/>
   <axis xyz="0.0 -1.0 -0.0"/>
-  <limit upper="0.008" lower="0.0" effort="100" velocity="5"/>
+  <limit upper="0.008" lower="0.0" effort="100" velocity="6.5"/>
 </joint>
 </robot>

File: minima/ros1_pump/urdf_minima_pump_description/urdf/urdf_minima_pump.xacro (robot description, xacro)
@@ -129,5 +129,5 @@
   <child link="Joint1_v4_1"/>
   <axis xyz="0.0 -0.0 1.0"/>
-  <limit upper="1.570796" lower="-1.570796" effort="100" velocity="10"/>
+  <limit upper="1.570796" lower="-1.570796" effort="100" velocity="6.5"/>
 </joint>
 <joint name="Revolute2" type="revolute">
@@ -136,5 +136,5 @@
   <child link="Joint2_v4_1"/>
   <axis xyz="0.0 1.0 0.0"/>
-  <limit upper="2.96706" lower="0.0" effort="100" velocity="10"/>
+  <limit upper="2.96706" lower="0.0" effort="100" velocity="6.5"/>
 </joint>
 <joint name="Revolute3" type="revolute">
@@ -143,5 +143,5 @@
   <child link="Joint3_v5_1"/>
   <axis xyz="0.0 1.0 0.0"/>
-  <limit upper="6.283185" lower="4.18879" effort="100" velocity="10"/>
+  <limit upper="6.283185" lower="4.18879" effort="100" velocity="6.5"/>
 </joint>
 <joint name="Revolute4" type="revolute">
@@ -150,5 +150,5 @@
   <child link="Joint4_p_v2_1"/>
   <axis xyz="-0.0 1.0 0.0"/>
-  <limit upper="1.570796" lower="-1.570796" effort="100" velocity="10"/>
+  <limit upper="1.570796" lower="-1.570796" effort="100" velocity="6.5"/>
 </joint>
 <joint name="Rigid5" type="fixed">

File: minima/ros2_gripper/urdf_minima_description/urdf/urdf_minima.xacro (robot description, xacro)
@@ -149,5 +149,5 @@
   <child link="Joint1_v4_1"/>
   <axis xyz="0.0 -0.0 1.0"/>
-  <limit upper="1.570796" lower="-1.570796" effort="100" velocity="10"/>
+  <limit upper="1.570796" lower="-1.570796" effort="100" velocity="6.5"/>
 </joint>
 <joint name="Revolute2" type="revolute">
@@ -156,5 +156,5 @@
   <child link="Joint2_v4_1"/>
   <axis xyz="0.0 1.0 0.0"/>
-  <limit upper="2.96706" lower="0.0" effort="100" velocity="10"/>
+  <limit upper="2.96706" lower="0.0" effort="100" velocity="6.5"/>
 </joint>
 <joint name="Revolute3" type="revolute">
@@ -163,5 +163,5 @@
   <child link="Joint3_v5_1"/>
   <axis xyz="0.0 1.0 0.0"/>
-  <limit upper="6.283185" lower="4.18879" effort="100" velocity="10"/>
+  <limit upper="6.283185" lower="4.18879" effort="100" velocity="6.5"/>
 </joint>
 <joint name="Revolute4" type="revolute">
@@ -170,5 +170,5 @@
   <child link="Joint4_v2_1"/>
   <axis xyz="-0.0 1.0 0.0"/>
-  <limit upper="1.570796" lower="-1.570796" effort="100" velocity="10"/>
+  <limit upper="1.570796" lower="-1.570796" effort="100" velocity="6.5"/>
 </joint>
 <joint name="Slider5" type="prismatic">

File: minima/ros2_pump/urdf_minima_pump_description/urdf/urdf_minima_pump.xacro (robot description, xacro)
@@ -129,5 +129,5 @@
   <child link="Joint1_v4_1"/>
   <axis xyz="0.0 -0.0 1.0"/>
-  <limit upper="1.570796" lower="-1.570796" effort="100" velocity="10"/>
+  <limit upper="1.570796" lower="-1.570796" effort="100" velocity="6.5"/>
 </joint>
 <joint name="Revolute2" type="revolute">
@@ -136,5 +136,5 @@
   <child link="Joint2_v4_1"/>
   <axis xyz="0.0 1.0 0.0"/>
-  <limit upper="2.96706" lower="0.0" effort="100" velocity="10"/>
+  <limit upper="2.96706" lower="0.0" effort="100" velocity="6.5"/>
 </joint>
 <joint name="Revolute3" type="revolute">
@@ -143,5 +143,5 @@
   <child link="Joint3_v5_1"/>
   <axis xyz="0.0 1.0 0.0"/>
-  <limit upper="6.283185" lower="4.18879" effort="100" velocity="10"/>
+  <limit upper="6.283185" lower="4.18879" effort="100" velocity="6.5"/>
 </joint>
 <joint name="Revolute4" type="revolute">
@@ -150,5 +150,5 @@
   <child link="Joint4_p_v2_1"/>
   <axis xyz="-0.0 1.0 0.0"/>
-  <limit upper="1.570796" lower="-1.570796" effort="100" velocity="10"/>
+  <limit upper="1.570796" lower="-1.570796" effort="100" velocity="6.5"/>
 </joint>
 <joint name="Rigid5" type="fixed">

File: minima_pro/ros1_gripper/urdf_minima_description/urdf/_converted.urdf (robot description, URDF)
Before this commit: robot urdf_minima, 7 links, 6 joints
Links:
- link Joint1_1: geometry collision mesh filename=file://C:/Users/dayueyue/Desktop/minima/src/assets/urdf/min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 scale=0.001 0.001 0.001; visual mesh filename=file://C:/Users/dayueyue/Desktop/minima/src/assets/urdf/min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 scale=0.001 0.001 0.001
- link Joint2_1: geometry collision mesh filename=file://C:/Users/dayueyue/Desktop/minima/src/assets/urdf/min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 scale=0.001 0.001 0.001; visual mesh filename=file://C:/Users/dayueyue/Desktop/minima/src/assets/urdf/min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 scale=0.001 0.001 0.001
- link Joint3_1: geometry collision mesh filename=file://C:/Users/dayueyue/Desktop/minima/src/assets/urdf/min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 scale=0.001 0.001 0.001; visual mesh filename=file://C:/Users/dayueyue/Desktop/minima/src/assets/urdf/min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 scale=0.001 0.001 0.001
- link Joint4_1: geometry collision mesh filename=file://C:/Users/dayueyue/Desktop/minima/src/assets/urdf/min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 scale=0.001 0.001 0.001; visual mesh filename=file://C:/Users/dayueyue/Desktop/minima/src/assets/urdf/min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 scale=0.001 0.001 0.001
- link Left_jaw_1: geometry collision mesh filename=file://C:/Users/dayueyue/Desktop/minima/src/assets/urdf/min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 scale=0.001 0.001 0.001; visual mesh filename=file://C:/Users/dayueyue/Desktop/minima/src/assets/urdf/min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 scale=0.001 0.001 0.001
- link Right_jaw_1: geometry collision mesh filename=file://C:/Users/dayueyue/Desktop/minima/src/assets/urdf/min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 scale=0.001 0.001 0.001; visual mesh filename=file://C:/Users/dayueyue/Desktop/minima/src/assets/urdf/min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 scale=0.001 0.001 0.001
- link base_link: geometry collision mesh filename=file://C:/Users/dayueyue/Desktop/minima/src/assets/urdf/min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 scale=0.001 0.001 0.001; visual mesh filename=file://C:/Users/dayueyue/Desktop/minima/src/assets/urdf/min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 scale=0.001 0.001 0.001

File: minima_pro/ros1_gripper/urdf_minima_description/urdf/urdf_minima.xacro (robot description, xacro)
@@ -149,5 +149,5 @@
   <child link="Joint1_1"/>
   <axis xyz="0.0 -0.0 1.0"/>
-  <limit upper="1.570796" lower="-1.570796" effort="100" velocity="100"/>
+  <limit upper="1.570796" lower="-1.570796" effort="100" velocity="6.5"/>
 </joint>
 <joint name="Revolute2" type="revolute">
@@ -156,5 +156,5 @@
   <child link="Joint2_1"/>
   <axis xyz="0.0 1.0 0.0"/>
-  <limit upper="2.96706" lower="0.0" effort="100" velocity="100"/>
+  <limit upper="2.96706" lower="0.0" effort="100" velocity="6.5"/>
 </joint>
 <joint name="Revolute3" type="revolute">
@@ -163,5 +163,5 @@
   <child link="Joint3_1"/>
   <axis xyz="-0.0 1.0 0.0"/>
-  <limit upper="6.283185" lower="4.18879" effort="100" velocity="100"/>
+  <limit upper="6.283185" lower="4.18879" effort="100" velocity="6.5"/>
 </joint>
 <joint name="Revolute4" type="revolute">
@@ -170,5 +170,5 @@
   <child link="Joint4_1"/>
   <axis xyz="-0.0 1.0 0.0"/>
-  <limit upper="1.570796" lower="-1.570796" effort="100" velocity="100"/>
+  <limit upper="1.570796" lower="-1.570796" effort="100" velocity="6.5"/>
 </joint>
 <joint name="Slider5" type="prismatic">
@@ -177,5 +177,5 @@
   <child link="Left_jaw_1"/>
   <axis xyz="0.0 1.0 0.0"/>
-  <limit upper="0.008" lower="0.0" effort="100" velocity="100"/>
+  <limit upper="0.008" lower="0.0" effort="100" velocity="6.5"/>
 </joint>
 <joint name="Slider6" type="prismatic">
@@ -184,5 +184,5 @@
   <child link="Right_jaw_1"/>
   <axis xyz="-0.0 -1.0 -0.0"/>
-  <limit upper="0.008" lower="0.0" effort="100" velocity="100"/>
+  <limit upper="0.008" lower="0.0" effort="100" velocity="6.5"/>
 </joint>
 </robot>

File: minima_pro/ros1_pump/urdf_minima_pump_description/urdf/urdf_minima_pump.xacro (robot description, xacro)
@@ -129,5 +129,5 @@
   <child link="Joint1_1"/>
   <axis xyz="0.0 -0.0 1.0"/>
-  <limit upper="1.570796" lower="-1.570796" effort="100" velocity="100"/>
+  <limit upper="1.570796" lower="-1.570796" effort="100" velocity="6.5"/>
 </joint>
 <joint name="Revolute2" type="revolute">
@@ -136,5 +136,5 @@
   <child link="Joint2_1"/>
   <axis xyz="0.0 1.0 0.0"/>
-  <limit upper="2.96706" lower="0.0" effort="100" velocity="100"/>
+  <limit upper="2.96706" lower="0.0" effort="100" velocity="6.5"/>
 </joint>
 <joint name="Revolute3" type="revolute">
@@ -143,5 +143,5 @@
   <child link="Joint3_1"/>
   <axis xyz="-0.0 1.0 0.0"/>
-  <limit upper="6.283185" lower="4.18879" effort="100" velocity="100"/>
+  <limit upper="6.283185" lower="4.18879" effort="100" velocity="6.5"/>
 </joint>
 <joint name="Revolute4" type="revolute">
@@ -150,5 +150,5 @@
   <child link="Joint4_1"/>
   <axis xyz="-0.0 1.0 0.0"/>
-  <limit upper="1.570796" lower="-1.570796" effort="100" velocity="100"/>
+  <limit upper="1.570796" lower="-1.570796" effort="100" velocity="6.5"/>
 </joint>
 <joint name="Rigid5" type="fixed">

File: minima_pro/ros2_gripper/urdf_minima_description/urdf/urdf_minima.xacro (robot description, xacro)
@@ -149,5 +149,5 @@
   <child link="Joint1_1"/>
   <axis xyz="0.0 -0.0 1.0"/>
-  <limit upper="1.570796" lower="-1.570796" effort="100" velocity="100"/>
+  <limit upper="1.570796" lower="-1.570796" effort="100" velocity="6.5"/>
 </joint>
 <joint name="Revolute2" type="revolute">
@@ -156,5 +156,5 @@
   <child link="Joint2_1"/>
   <axis xyz="0.0 1.0 0.0"/>
-  <limit upper="2.96706" lower="0.0" effort="100" velocity="100"/>
+  <limit upper="2.96706" lower="0.0" effort="100" velocity="6.5"/>
 </joint>
 <joint name="Revolute3" type="revolute">
@@ -163,5 +163,5 @@
   <child link="Joint3_1"/>
   <axis xyz="-0.0 1.0 0.0"/>
-  <limit upper="6.283185" lower="4.18879" effort="100" velocity="100"/>
+  <limit upper="6.283185" lower="4.18879" effort="100" velocity="6.5"/>
 </joint>
 <joint name="Revolute4" type="revolute">
@@ -170,5 +170,5 @@
   <child link="Joint4_1"/>
   <axis xyz="-0.0 1.0 0.0"/>
-  <limit upper="1.570796" lower="-1.570796" effort="100" velocity="100"/>
+  <limit upper="1.570796" lower="-1.570796" effort="100" velocity="6.5"/>
 </joint>
 <joint name="Slider5" type="prismatic">
@@ -177,5 +177,5 @@
   <child link="Left_jaw_1"/>
   <axis xyz="0.0 1.0 0.0"/>
-  <limit upper="0.008" lower="0.0" effort="100" velocity="100"/>
+  <limit upper="0.008" lower="0.0" effort="100" velocity="6.5"/>
 </joint>
 <joint name="Slider6" type="prismatic">
@@ -184,5 +184,5 @@
   <child link="Right_jaw_1"/>
   <axis xyz="-0.0 -1.0 -0.0"/>
-  <limit upper="0.008" lower="0.0" effort="100" velocity="100"/>
+  <limit upper="0.008" lower="0.0" effort="100" velocity="6.5"/>
 </joint>
 </robot>

File: minima_pro/ros2_pump/urdf_minima_pump_description/urdf/urdf_minima_pump.xacro (robot description, xacro)
@@ -129,5 +129,5 @@
   <child link="Joint1_1"/>
   <axis xyz="0.0 -0.0 1.0"/>
-  <limit upper="1.570796" lower="-1.570796" effort="100" velocity="100"/>
+  <limit upper="1.570796" lower="-1.570796" effort="100" velocity="6.5"/>
 </joint>
 <joint name="Revolute2" type="revolute">
@@ -136,5 +136,5 @@
   <child link="Joint2_1"/>
   <axis xyz="0.0 1.0 0.0"/>
-  <limit upper="2.96706" lower="0.0" effort="100" velocity="100"/>
+  <limit upper="2.96706" lower="0.0" effort="100" velocity="6.5"/>
 </joint>
 <joint name="Revolute3" type="revolute">
@@ -143,5 +143,5 @@
   <child link="Joint3_1"/>
   <axis xyz="-0.0 1.0 0.0"/>
-  <limit upper="6.283185" lower="4.18879" effort="100" velocity="100"/>
+  <limit upper="6.283185" lower="4.18879" effort="100" velocity="6.5"/>
 </joint>
 <joint name="Revolute4" type="revolute">
@@ -150,5 +150,5 @@
   <child link="Joint4_1"/>
   <axis xyz="-0.0 1.0 0.0"/>
-  <limit upper="1.570796" lower="-1.570796" effort="100" velocity="100"/>
+  <limit upper="1.570796" lower="-1.570796" effort="100" velocity="6.5"/>
 </joint>
 <joint name="Rigid5" type="fixed">
